Commit message: feature: ssmr shape change

File: urdf/skid_steer_bot.xacro (robot description, xacro)
@@ -7,5 +7,5 @@
   <xacro:property name="mower_width" value="${scale * 0.46}" />
   <xacro:property name="mower_length" value="${scale * 0.46}" />
-  <xacro:property name="mower_height" value="${scale * 0.3}" />
+  <xacro:property name="mower_height" value="${scale * 0.25}" />
   <xacro:property name="mower_mass" value="${scale * 10}" />
   <xacro:property name="base_x_offset" value="0" />
@@ -21,6 +21,6 @@
   <xacro:property name="mower_frame_width" value="${mower_width - 2.1 * wheel_length}" />
   <xacro:property name="mower_frame_length" value="${mower_length*1.2}" />
-  <xacro:property name="mower_frame_height" value="${mower_height/4.0}" />
-  <xacro:property name="hardware_width" value="${mower_width/2.0}" />
+  <xacro:property name="mower_frame_height" value="${mower_height}" />
+  <xacro:property name="hardware_width" value="${mower_frame_width}" />
   <xacro:property name="hardware_length" value="${mower_length/2.0}" />
   <xacro:property name="hardware_height" value="${mower_height/2.0}" />
@@ -32,14 +32,15 @@
   <xacro:property name="wheel_x_offset" value="${base_x_offset + mower_length/2.0}" />
   <xacro:property name="wheel_y_offset" value="${mower_width/2.0 - wheel_length/2.0}" />
+  <xacro:property name="wheel_z_offset" value="${6.0*mower_height/15.0}" />
   <xacro:property name="camerra_width" value="0.05" />
   <xacro:property name="camerra_length" value="0.05" />
   <xacro:property name="camerra_height" value="0.05" />
-  <xacro:property name="camerra_x_offset" value="${hardware_length/2.0 + base_x_offset - camerra_length/2.0 + 0.001}" />
-  <xacro:property name="camerra_z_offset" value="${hardware_height - camerra_height/2.0 + 0.001}" />
+  <xacro:property name="camerra_x_offset" value="${mower_frame_length/2.0 + base_x_offset - camerra_length/2.0 + 0.001}" />
+  <xacro:property name="camerra_z_offset" value="${mower_frame_height/2.0 - 2.5*camerra_height + 0.001 }" />
   <xacro:property name="laser_width" value="0.1" />
   <xacro:property name="laser_length" value="0.1" />
   <xacro:property name="laser_height" value="0.1" />
-  <xacro:property name="laser_x_offset" value="${base_x_offset}" />
-  <xacro:property name="laser_z_offset" value="${hardware_height + 0.025}" />
+  <xacro:property name="laser_x_offset" value="${2.0*laser_width + mower_frame_height/2.0 + base_x_offset - 0.025}" />
+  <xacro:property name="laser_z_offset" value="${mower_frame_height/2.0 + 0.1 - laser_height}" />
   <xacro:property name="wheel_kp" value="1000000.0" />
   <xacro:property name="wheel_kd" value="100.0" />
@@ -76,5 +77,5 @@
     </visual>
     <!-- blade frame -->
-    <collision>
+    <!-- <collision>
       <origin xyz="${base_x_offset} 0 0" rpy=" 0 0 0"/>
       <geometry>
@@ -87,7 +88,7 @@
         <cylinder radius="${mower_width/2.0}" length="${mower_frame_height}"/>
       </geometry>
-    </visual>
+    </visual> -->
     <!-- hardware frame -->
-    <collision>
+    <!-- <collision>
       <origin xyz="${base_x_offset} 0 ${hardware_z_offset}" rpy=" 0 0 0"/>
       <geometry>
@@ -100,9 +101,9 @@
         <box size="${hardware_length} ${hardware_width} ${hardware_height}"/>
       </geometry>
-    </visual>
+    </visual> -->
   </link>
   <!-- left back wheel -->
   <joint type="continuous" name="left_back_wheel_hinge">
-    <origin xyz="-${wheel_x_offset} ${wheel_y_offset} 0" rpy="0 0 0"/>
+    <origin xyz="-${wheel_x_offset} ${wheel_y_offset} -${wheel_z_offset}" rpy="0 0 0"/>
     <child link="left_back_wheel"/>
     <parent link="chassis"/>
@@ -146,5 +147,5 @@
   <!-- right back wheel -->
   <joint type="continuous" name="right_back_wheel_hinge">
-    <origin xyz="-${wheel_x_offset} -${wheel_y_offset} 0" rpy="0 0 0"/>
+    <origin xyz="-${wheel_x_offset} -${wheel_y_offset} -${wheel_z_offset}" rpy="0 0 0"/>
     <child link="right_back_wheel"/>
     <parent link="chassis"/>
@@ -188,5 +189,5 @@
   <!-- left front wheel -->
   <joint type="continuous" name="left_front_wheel_hinge">
-    <origin xyz="${wheel_x_offset} ${wheel_y_offset} 0" rpy="0 0 0"/>
+    <origin xyz="${wheel_x_offset} ${wheel_y_offset} -${wheel_z_offset}" rpy="0 0 0"/>
     <child link="left_front_wheel"/>
     <parent link="chassis"/>
@@ -230,5 +231,5 @@
   <!-- right front wheel -->
   <joint type="continuous" name="right_front_wheel_hinge">
-    <origin xyz="${wheel_x_offset} -${wheel_y_offset} 0" rpy="0 0 0"/>
+    <origin xyz="${wheel_x_offset} -${wheel_y_offset} -${wheel_z_offset}" rpy="0 0 0"/>
     <child link="right_front_wheel"/>
     <parent link="chassis"/>

Commit message: feature: initial position

File: urdf/skid_steer_bot.xacro (robot description, xacro)
@@ -51,5 +51,5 @@
   <link name="robot_footprint"></link>
   <joint name="robot_footprint_joint" type="fixed">
-    <origin xyz="0 0 0" rpy="0 0 0" />
+    <origin xyz="-1.0 -1.0 0" rpy="0 0 0" />
     <parent link="robot_footprint" />
     <child link="chassis" />

Commit message: feat: adding 3 cameras to robot

File: urdf/skid_steer_bot.xacro (robot description, xacro)
@@ -24,8 +24,8 @@
   <xacro:property name="hardware_width" value="${mower_width/2.0}" />
   <xacro:property name="hardware_length" value="${mower_length/2.0}" />
-  <xacro:property name="hardware_height" value="${mower_height/2.0}" />
+  <xacro:property name="hardware_height" value="${mower_height/2.0 + 0.1}" />
   <xacro:property name="hardware_z_offset" value="${hardware_height/2.0}" />
   <xacro:property name="wheel_length" value="${scale * 0.05}" />
-  <xacro:property name="wheel_radius" value="${scale * 0.08}" />
+  <xacro:property name="wheel_radius" value="${scale * 0.11}" />
   <xacro:property name="wheel_mass" value="${scale * 1}" />
   <xacro:property name="wheel_inertia" value="${scale * 1e-3}" />
@@ -35,6 +35,13 @@
   <xacro:property name="camerra_length" value="0.05" />
   <xacro:property name="camerra_height" value="0.05" />
-  <xacro:property name="camerra_x_offset" value="${hardware_length/2.0 + base_x_offset - camerra_length/2.0 + 0.001}" />
-  <xacro:property name="camerra_z_offset" value="${hardware_height - camerra_height/2.0 + 0.001}" />
+  <xacro:property name="camerra_x_offset" value="${hardware_length/2.0 + base_x_offset - camerra_length/2.0 + 0.02}" />
+  <xacro:property name="camerra_z_offset" value="${hardware_height - camerra_height/2.0 + 0.01}" />
+  <xacro:property name="camerra_left_x_offset" value="${hardware_length/2.0 + base_x_offset - camerra_length/2.0 + 0.02}" />
+  <xacro:property name="camerra_left_z_offset" value="${hardware_height - camerra_height/2.0 + 0.01}" />
+  <xacro:property name="camerra_left_y_offset" value="${scale * 0.1}" />
+  <xacro:property name="side_camera_yaw" value="0.2618" />
+  <xacro:property name="camerra_right_x_offset" value="${hardware_length/2.0 + base_x_offset - camerra_length/2.0 + 0.02}" />
+  <xacro:property name="camerra_right_z_offset" value="${hardware_height - camerra_height/2.0 + 0.01}" />
+  <xacro:property name="camerra_right_y_offset" value="${scale * -0.1}" />
   <xacro:property name="laser_width" value="0.1" />
   <xacro:property name="laser_length" value="0.1" />
@@ -272,5 +279,5 @@
   <link name='camera'>
     <inertial>
-      <mass value="0.1"/>
+      <mass value="0.001"/>
       <origin xyz="0 0 0" rpy=" 0 0 0"/>
       <inertia
@@ -300,4 +307,64 @@
     <joint_properties damping="1.0" friction="1.0"/>
   </joint>
+  <link name='camera_left'>
+    <inertial>
+      <mass value="0.001"/>
+      <origin xyz="0 0 0" rpy=" 0 0 0"/>
+      <inertia
+          ixx="1e-6" ixy="0" ixz="0"
+          iyy="1e-6" iyz="0"
+          izz="1e-6"/>
+    </inertial>
+    <collision name='camera_left_collision'>
+      <origin xyz="0 0 0" rpy=" 0 0 0"/>
+      <geometry>
+        <box size="${camerra_length} ${camerra_width} ${camerra_height}"/>
+      </geometry>
+    </collision>
+    <visual name='camera_visual'>
+      <origin xyz="0 0 0" rpy=" 0 0 0"/>
+      <geometry>
+        <box size="${camerra_length} ${camerra_width} ${camerra_height}"/>
+      </geometry>
+    </visual>
+  </link>
+  <joint type="fixed" name="camera_left_joint">
+    <origin xyz="${camerra_left_x_offset} ${camerra_left_y_offset} ${camerra_left_z_offset}" rpy="0 0 ${side_camera_yaw}"/>
+    <child link="camera_left"/>
+    <parent link="chassis"/>
+    <axis xyz="0 1 0" rpy="0 0 0"/>
+    <limit effort="10000" velocity="1000"/>
+    <joint_properties damping="1.0" friction="1.0"/>
+  </joint>
+  <link name='camera_right'>
+    <inertial>
+      <mass value="0.001"/>
+      <origin xyz="0 0 0" rpy=" 0 0 0"/>
+      <inertia
+          ixx="1e-6" ixy="0" ixz="0"
+          iyy="1e-6" iyz="0"
+          izz="1e-6"/>
+    </inertial>
+    <collision name='camera_right_collision'>
+      <origin xyz="0 0 0" rpy=" 0 0 0"/>
+      <geometry>
+        <box size="${camerra_length} ${camerra_width} ${camerra_height}"/>
+      </geometry>
+    </collision>
+    <visual name='camera_visual'>
+      <origin xyz="0 0 0" rpy=" 0 0 0"/>
+      <geometry>
+        <box size="${camerra_length} ${camerra_width} ${camerra_height}"/>
+      </geometry>
+    </visual>
+  </link>
+  <joint type="fixed" name="camera_right_joint">
+    <origin xyz="${camerra_right_x_offset} ${camerra_right_y_offset} ${camerra_right_z_offset}" rpy="0 0 ${-side_camera_yaw}"/>
+    <child link="camera_right"/>
+    <parent link="chassis"/>
+    <axis xyz="0 1 0" rpy="0 0 0"/>
+    <limit effort="10000" velocity="1000"/>
+    <joint_properties damping="1.0" friction="1.0"/>
+  </joint>
   <link name='hokuyo'>
     <pose>0 0 0 0 0 0</pose>

Commit message: feat: city simulation for skid steered mobile robot

File: urdf/skid_steer_bot.xacro (robot description, xacro)
@@ -40,5 +40,5 @@
   <xacro:property name="camerra_left_z_offset" value="${hardware_height - camerra_height/2.0 + 0.01}" />
   <xacro:property name="camerra_left_y_offset" value="${scale * 0.1}" />
-  <xacro:property name="side_camera_yaw" value="0.2618" />
+  <xacro:property name="side_camera_yaw" value="0.523" />
   <xacro:property name="camerra_right_x_offset" value="${hardware_length/2.0 + base_x_offset - camerra_length/2.0 + 0.02}" />
   <xacro:property name="camerra_right_z_offset" value="${hardware_height - camerra_height/2.0 + 0.01}" />

Commit message: feat: simulation working with ros1_bridge for ros2

File: urdf/skid_steer_bot.xacro (robot description, xacro)
@@ -308,5 +308,5 @@
     <joint_properties damping="1.0" friction="1.0"/>
   </joint>
-  <link name='camera_left'>
+  <!-- <link name='camera_left'>
     <inertial>
       <mass value="0.001"/>
@@ -367,5 +367,5 @@
     <limit effort="10000" velocity="1000"/>
     <joint_properties damping="1.0" friction="1.0"/>
-  </joint>
+  </joint> -->
   <link name='hokuyo'>
     <pose>0 0 0 0 0 0</pose>
